File: EnvKB65.kicad_pcb (KiCad board)
At the start: 2 copper layers, 326.8 x 94.7 mm, 148 parts, among them U1 Pico

Commit message: slimmed design down a bit at the cost of some keys
Parts:
- removed D_14, D_30, D_45: D, Diode_SMD:D_SOD-123
- removed K_14, K_30, K_45: KEYSW, MX_Only:MXOnly-1U-NoLED
- K_29: footprint MX_Only:MXOnly-ISO-ROTATED-ReversedStabilizers -> MX_Only:MXOnly-ISO-ROTATED-ReversedStabilizers-NoLED
- moved D_75 16.6 mm to (368.8, 190.2)
- moved D_62 16.3 mm to (369.2, 175.7)
- moved U1 9.43 mm to (367.8, 127.0)
- moved Ref** 9.23 mm to (367.8, 156.7)
Connections:
- net row5 renamed Net-(U1-Pad34)
- net vbus renamed Net-(U1-Pad40)
- U1 pad 1: col16 -> col0
- U1 pad 10: col11 -> col7
- U1 pad 11: col10 -> col8
- U1 pad 14: col9 -> col10
- U1 pad 15: col8 -> col11
- U1 pad 16: col7 -> col12
- U1 pad 17: col6 -> col13
- U1 pad 19: col5 -> col14
- U1 pad 2: col15 -> col1
- U1 pad 20: col4 -> col15
- U1 pad 21: col3 -> col16
- U1 pad 22: col2 -> Net-(U1-Pad22)
- U1 pad 23: gnd -> gnds
- U1 pad 24: col1 -> Net-(U1-Pad24)
- U1 pad 25: col0 -> Net-(U1-Pad25)
- U1 pad 26: row0 -> Net-(U1-Pad26)
- U1 pad 27: row1 -> Net-(U1-Pad27)
- U1 pad 29: row2 -> Net-(U1-Pad29)
- U1 pad 31: row3 -> Net-(U1-Pad31)
- U1 pad 32: row4 -> Net-(U1-Pad32)
- U1 pad 33: Net-(U1-Pad33) -> gnd
- U1 pad 4: col14 -> col2
- U1 pad 5: col13 -> col3
- U1 pad 6: col12 -> col4
- U1 pad 7: col13 -> col5
- U1 pad 9: col12 -> col6
Routing:
- net col0: track 82.2 -> 378.0 mm
- net col1: track 79.2 -> 356.0 mm
- net col2: track 67.4 -> 326.7 mm
- net col3: track 92.9 -> 333.7 mm
- net col4: track 88.0 -> 310.2 mm
- net col5: track 67.5 -> 279.0 mm
- net col6: track 87.5 -> 284.6 mm
- net col7: track 67.6 -> 247.0 mm
- net col8: track 87.2 -> 245.5 mm
- net col9: track 67.9 -> 207.4 mm
- net col10: track 89.4 -> 222.2 mm
- net col11: track 88.3 -> 200.3 mm
- net col13: track 64.7 -> 158.3 mm
- net col12: track 96.5 -> 188.0 mm
- net row0: track 271.7 -> 324.3 mm
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- removed copper zone on B.Cu, net gnd
- removed copper zone on F.Cu, net gnd
Other:
- board outline removed

Commit message: Routed Traces, Add Mounting holes and edge cuts
Parts:
- added H1: MountingHole, MountingHole:MountingHole_2.2mm_M2, F.Cu at (382.2, 101.0)
- added H2: MountingHole, MountingHole:MountingHole_2.2mm_M2, F.Cu at (69.0, 101.0)
- added H3: MountingHole, MountingHole:MountingHole_2.2mm_M2, F.Cu at (68.8, 178.2)
- added H4: MountingHole, MountingHole:MountingHole_2.2mm_M2, F.Cu at (367.8, 180.5)
- added H5: MountingHole, MountingHole:MountingHole_2.2mm_M2, F.Cu at (225.0, 122.5)
- added H6: MountingHole, MountingHole:MountingHole_2.2mm_M2, F.Cu at (231.2, 178.0)
- Ref**: footprint MechboardsLogo:mechboardsLOGO_10mm -> MechboardsLogo:mechboardsLOGO_20mm
- moved U1 3.87 mm to (367.8, 123.2)
- moved Ref** 2.83 mm to (367.8, 153.9)
Connections:
- U1 pad 22: Net-(U1-Pad22) -> row4
- U1 pad 23: gnds -> gnd
- U1 pad 24: Net-(U1-Pad24) -> row3
- U1 pad 25: Net-(U1-Pad25) -> row2
- U1 pad 26: Net-(U1-Pad26) -> row1
- U1 pad 27: Net-(U1-Pad27) -> row0
Routing:
- net row0: track 324.3 -> 353.5 mm
- net row1: track 301.0 -> 327.0 mm
- net row2: track 287.6 -> 309.6 mm
- net row3: track 323.1 -> 342.6 mm
- net row4: track 337.8 -> 352.0 mm
- net col10: track 222.2 -> 211.1 mm
- net col11: track 200.3 -> 192.1 mm
- net col12: track 188.0 -> 181.8 mm
- net col13: track 158.3 -> 153.1 mm
- net col6: track 284.6 -> 280.2 mm
- net col16: track 36.3 -> 40.1 mm
- net col15: track 37.0 -> 40.8 mm
- net col7: track 247.0 -> 244.2 mm
- net gnd: track 0.00 -> 2.59 mm
- net col8: track 245.5 -> 243.2 mm
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- added copper zone on B.Cu, net gnd
- added copper zone on F.Cu, net gnd
Other:
- board outline added: 319.4 x 99.3 mm

Commit message: Final Adjustments And Gerber Creation for Revision0
Parts:
- moved H3 1.80 mm to (70.6, 178.2)
- moved Ref** 0.19 mm to (367.6, 153.9)
Routing:
- net col0: track 378.0 -> 380.4 mm
Other:
- board text added: "USB"
- board text added: "http://Mechboards.co.uk"
- board text added: "https://github.com/Envious-Data/Env-KB65M"
Changed lines of the file:
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@@
   (general
     (thickness 1.6)
-    (drawings 11)
-    (tracks 620)
+    (drawings 15)
+    (tracks 624)
     (zones 0)
     (modules 148)
@@
       (outputformat 1)
       (mirror false)
-      (drillshape 1)
+      (drillshape 0)
       (scaleselection 1)
-      (outputdirectory ""))
+      (outputdirectory "_gerber/"))
   )
   (net 0 "")
@@
       (effects (font (size 1 1) (thickness 0.15)))
     )
+    (fp_circle (center 0 0) (end 2.2 0) (layer Cmts.User) (width 0.15))
+    (fp_circle (center 0 0) (end 2.45 0) (layer F.CrtYd) (width 0.05))
     (fp_text user %R (at 0.3 0) (layer F.Fab)
       (effects (font (size 1 1) (thickness 0.15)))
     )
-    (fp_circle (center 0 0) (end 2.2 0) (layer Cmts.User) (width 0.15))
-    (fp_circle (center 0 0) (end 2.45 0) (layer F.CrtYd) (width 0.05))
     (pad 1 np_thru_hole circle (at 0 0) (size 2.2 2.2) (drill 2.2) (layers *.Cu *.Mask))
   )
@@
     (tags "mounting hole 2.2mm no annular m2")
     (attr virtual)
-    (fp_text reference H5 (at 0 -3.2) (layer F.SilkS)
+    (fp_text reference H5 (at 0 -3.2) (layer Dwgs.User)
       (effects (font (size 1 1) (thickness 0.15)))
     )
@@
       (effects (font (size 1 1) (thickness 0.15)))
     )
+    (fp_circle (center 0 0) (end 2.2 0) (layer Cmts.User) (width 0.15))
+    (fp_circle (center 0 0) (end 2.45 0) (layer F.CrtYd) (width 0.05))
     (fp_text user %R (at 0.3 0) (layer F.Fab)
       (effects (font (size 1 1) (thickness 0.15)))
     )
-    (fp_circle (center 0 0) (end 2.2 0) (layer Cmts.User) (width 0.15))
-    (fp_circle (center 0 0) (end 2.45 0) (layer F.CrtYd) (width 0.05))
     (pad 1 np_thru_hole circle (at 0 0) (size 2.2 2.2) (drill 2.2) (layers *.Cu *.Mask))
   )
@@
       (effects (font (size 1 1) (thickness 0.15)))
     )
+    (fp_circle (center 0 0) (end 2.2 0) (layer Cmts.User) (width 0.15))
+    (fp_circle (center 0 0) (end 2.45 0) (layer F.CrtYd) (width 0.05))
     (fp_text user %R (at 0.3 0) (layer F.Fab)
       (effects (font (size 1 1) (thickness 0.15)))
     )
-    (fp_circle (center 0 0) (end 2.2 0) (layer Cmts.User) (width 0.15))
-    (fp_circle (center 0 0) (end 2.45 0) (layer F.CrtYd) (width 0.05))
     (pad 1 np_thru_hole circle (at 0 0) (size 2.2 2.2) (drill 2.2) (layers *.Cu *.Mask))
   )
   (module MountingHole:MountingHole_2.2mm_M2 (layer F.Cu)
-    (at 68.8 178.2)
+    (at 70.6 178.2)
     (descr "Mounting Hole 2.2mm, no annular, M2")
     (tags "mounting hole 2.2mm no annular m2")
@@
       (effects (font (size 1 1) (thickness 0.15)))
     )
+    (fp_circle (center 0 0) (end 2.2 0) (layer Cmts.User) (width 0.15))
+    (fp_circle (center 0 0) (end 2.45 0) (layer F.CrtYd) (width 0.05))
     (fp_text user %R (at 0.3 0) (layer F.Fab)
       (effects (font (size 1 1) (thickness 0.15)))
     )
-    (fp_circle (center 0 0) (end 2.2 0) (layer Cmts.User) (width 0.15))
-    (fp_circle (center 0 0) (end 2.45 0) (layer F.CrtYd) (width 0.05))
     (pad 1 np_thru_hole circle (at 0 0) (size 2.2 2.2) (drill 2.2) (layers *.Cu *.Mask))
   )
@@
       (effects (font (size 1 1) (thickness 0.15)))
     )
+    (fp_circle (center 0 0) (end 2.2 0) (layer Cmts.User) (width 0.15))
+    (fp_circle (center 0 0) (end 2.45 0) (layer F.CrtYd) (width 0.05))
     (fp_text user %R (at 0.3 0) (layer F.Fab)
       (effects (font (size 1 1) (thickness 0.15)))
     )
-    (fp_circle (center 0 0) (end 2.2 0) (layer Cmts.User) (width 0.15))
-    (fp_circle (center 0 0) (end 2.45 0) (layer F.CrtYd) (width 0.05))
     (pad 1 np_thru_hole circle (at 0 0) (size 2.2 2.2) (drill 2.2) (layers *.Cu *.Mask))
   )
@@
       (effects (font (size 1 1) (thickness 0.15)))
     )
+    (fp_circle (center 0 0) (end 2.2 0) (layer Cmts.User) (width 0.15))
+    (fp_circle (center 0 0) (end 2.45 0) (layer F.CrtYd) (width 0.05))
     (fp_text user %R (at 0.3 0) (layer F.Fab)
       (effects (font (size 1 1) (thickness 0.15)))
     )
-    (fp_circle (center 0 0) (end 2.2 0) (layer Cmts.User) (width 0.15))
-    (fp_circle (center 0 0) (end 2.45 0) (layer F.CrtYd) (width 0.05))
     (pad 1 np_thru_hole circle (at 0 0) (size 2.2 2.2) (drill 2.2) (layers *.Cu *.Mask))
   )
   (module MechboardsLogo:mechboardsLOGO_20mm locked (layer F.Cu)
-    (at 367.79 153.9)
+    (at 367.6 153.9)
     (fp_text reference Ref** (at -1.5 0) (layer F.SilkS) hide
       (effects (font (size 1.27 1.27) (thickness 0.15)))
@@
     (descr "Through hole straight pin header, 2x20, 2.54mm pitch, double rows")
     (tags "Through hole pin header THT 2x20 2.54mm double row")
-    (fp_text reference U1 (at 0 0) (layer F.SilkS)
+    (fp_text reference U1 (at 0 0) (layer Dwgs.User)
       (effects (font (size 1 1) (thickness 0.15)))
     )
@@
     )
   )
+  (gr_text USB (at 367.8 99.8) (layer F.SilkS)
+    (effects (font (size 1 1) (thickness 0.15)))
+  )
+  (gr_poly (pts (xy 368.4 99) (xy 367.2 99) (xy 367.8 98.4)) (layer F.SilkS) (width 0.1))
+  (gr_text https://github.com/Envious-Data/Env-KB65M (at 335.8 99) (layer B.SilkS)
+    (effects (font (size 1 1) (thickness 0.15)) (justify mirror))
+  )
+  (gr_text http://Mechboards.co.uk (at 74.6 100.2) (layer F.SilkS)
+    (effects (font (size 2 2) (thickness 0.175)) (justify left))
+  )
   (dimension 2 (width 0.12) (layer Dwgs.User)
     (gr_text "2.000 mm" (at 72.97 98.65 270) (layer Dwgs.User)
@@
   (segment (start 76.55 160.64957) (end 71.08045 166.11912) (width 0.25) (layer F.Cu) (net 1))
   (segment (start 76.55 147.74492) (end 76.55 160.64957) (width 0.25) (layer F.Cu) (net 1))
-  (segment (start 71.08045 166.11912) (end 71.675 166.71367) (width 0.25) (layer F.Cu) (net 1))
-  (segment (start 71.675 184.57457) (end 71.08045 185.16912) (width 0.25) (layer F.Cu) (net 1))
-  (segment (start 71.675 166.71367) (end 71.675 184.57457) (width 0.25) (layer F.Cu) (net 1))
   (segment (start 148.741342 101.44997) (end 150.491352 99.69996) (width 0.25) (layer B.Cu) (net 1))
   (segment (start 94.349098 101.44997) (end 148.741342 101.44997) (width 0.25) (layer B.Cu) (net 1))
@@
   (segment (start 345.05 100.95) (end 356.96 100.95) (width 0.25) (layer B.Cu) (net 1))
   (segment (start 343.79996 99.69996) (end 345.05 100.95) (width 0.25) (layer B.Cu) (net 1))
+  (segment (start 71.08045 185.16912) (end 74.6 181.64957) (width 0.25) (layer F.Cu) (net 1))
+  (segment (start 74.6 181.64957) (end 74.6 174) (width 0.25) (layer F.Cu) (net 1))
+  (segment (start 71.210451 166.249121) (end 71.08045 166.11912) (width 0.25) (layer F.Cu) (net 1))
+  (segment (start 71.210451 170.610451) (end 71.210451 166.249121) (width 0.25) (layer F.Cu) (net 1))
+  (segment (start 74.6 174) (end 71.210451 170.610451) (width 0.25) (layer F.Cu) (net 1))
   (segment (start 92.641701 166.249121) (end 92.5117 166.11912) (width 0.25) (layer F.Cu) (net 2))
   (segment (start 92.641701 182.917871) (end 92.641701 166.249121) (width 0.25) (layer F.Cu) (net 2))
@@
   (segment (start 212.25 142.98242) (end 212.25 128.69492) (width 0.25) (layer F.Cu) (net 9))
   (segment (start 216.3367 147.06912) (end 212.25 142.98242) (width 0.25) (layer F.Cu) (net 9))
-  (segment (start 217.627799 157.885219) (end 225.8617 166.11912) (width 0.25) (layer F.Cu) (net 9))
-  (segment (start 217.627799 150.098217) (end 217.627799 157.885219) (width 0.25) (layer F.Cu) (net 9))
-  (segment (start 216.3367 148.807118) (end 217.627799 150.098217) (width 0.25) (layer F.Cu) (net 9))
-  (segment (start 216.3367 147.06912) (end 216.3367 148.807118) (width 0.25) (layer F.Cu) (net 9))
   (segment (start 226.986699 183.912869) (end 228.24295 185.16912) (width 0.25) (layer F.Cu) (net 9))
   (segment (start 226.986699 167.244119) (end 226.986699 183.912869) (width 0.25) (layer F.Cu) (net 9))
@@
   (segment (start 358.89 124.42) (end 350.800752 124.42) (width 0.25) (layer F.Cu) (net 9))
   (segment (start 349.750047 116.353785) (end 349.750047 122.999953) (width 0.25) (layer F.Cu) (net 9))
+  (segment (start 217.4 157.65742) (end 225.8617 166.11912) (width 0.25) (layer F.Cu) (net 9))
+  (segment (start 217.4 151.2) (end 217.4 157.65742) (width 0.25) (layer F.Cu) (net 9))
+  (segment (start 216.8 150.6) (end 217.4 151.2) (width 0.25) (layer F.Cu) (net 9))
+  (segment (start 216.8 148.8) (end 216.8 150.6) (width 0.25) (layer F.Cu) (net 9))
+  (segment (start 216.3367 148.3367) (end 216.8 148.8) (width 0.25) (layer F.Cu) (net 9))
+  (segment (start 216.3367 147.06912) (end 216.3367 148.3367) (width 0.25) (layer F.Cu) (net 9))
   (segment (start 238.55821 108.96912) (end 240.1492 108.96912) (width 0.25) (layer F.Cu) (net 10))
   (segment (start 230.6242 116.90313) (end 238.55821 108.96912) (width 0.25) (layer F.Cu) (net 10))
@@
   (segment (start 231.915299 129.310219) (end 231.915299 143.597719) (width 0.25) (layer F.Cu) (net 10))
   (segment (start 230.6242 128.01912) (end 231.915299 129.310219) (width 0.25) (layer F.Cu) (net 10))
-  (segment (start 235.516701 147.199121) (end 235.3867 147.06912) (width 0.25) (layer F.Cu) (net 10))
-  (segment (start 235.516701 156.724121) (end 235.516701 147.199121) (width 0.25) (layer F.Cu) (net 10))
-  (segment (start 244.9117 166.11912) (end 235.516701 156.724121) (width 0.25) (layer F.Cu) (net 10))
   (segment (start 273.48075 104) (end 276.430759 101.049991) (width 0.25) (layer F.Cu) (net 10))
   (segment (start 245.118319 104.000001) (end 273.48075 104) (width 0.25) (layer F.Cu) (net 10))
@@
   (segment (start 351.26 126.96) (end 349.100041 124.800041) (width 0.25) (layer F.Cu) (net 10))
   (segment (start 358.89 126.96) (end 351.26 126.96) (width 0.25) (layer F.Cu) (net 10))
+  (segment (start 236 147.68242) (end 235.3867 147.06912) (width 0.25) (layer F.Cu) (net 10))
+  (segment (start 236 157.20742) (end 236 147.68242) (width 0.25) (layer F.Cu) (net 10))
+  (segment (start 244.9117 166.11912) (end 236 157.20742) (width 0.25) (layer F.Cu) (net 10))
   (segment (start 263.159698 166.11912) (end 263.9617 166.11912) (width 0.25) (layer F.Cu) (net 11))
   (segment (start 259.1992 170.079618) (end 263.159698 166.11912) (width 0.25) (layer F.Cu) (net 11))

Commit message: Changed Diodes to SOD-323 and separated Position files
Parts:
- D_0, D_1, D_10, D_11, D_12, D_13, D_16, D_17, D_18, D_19, D_2, D_20, D_21, D_22, D_23, D_24, D_25, D_26, D_27, D_28, D_29, D_3, D_32, D_33, D_34, D_35, D_36, D_37, D_38, D_39, D_4, D_40, D_41, D_42, D_43, D_44, D_47, D_48, D_49, D_5, D_50, D_51, D_52, D_53, D_54, D_55, D_56, D_57, D_58, D_59, D_6, D_60, D_61, D_62, D_63, D_64, D_65, D_66, D_67, D_68, D_69, D_7, D_70, D_71, D_72, D_73, D_74, D_75, D_8, D_9: footprint Diode_SMD:D_SOD-123 -> Diode_SMD:D_SOD-323_HandSoldering
