File: TopPCB/EnvKB65-SwitchPlate.sch (KiCad schematic (older format))
At the start: 159 parts, among them U1 Pico

Commit message: Mount hole tweak to allow for switches to seat properly with a spacer installed
Parts:
- removed D_0, D_1, D_10, D_11, D_12, D_13, D_14, D_15, D_16, D_17, D_18, D_19, D_2, D_20, D_21, D_22, D_23, D_24, D_25, D_26, D_27, D_28, D_29, D_3, D_30, D_31, D_32, D_33, D_34, D_35, D_36, D_37, D_38, D_39, D_4, D_40, D_41, D_42, D_43, D_44, D_45, D_46, D_47, D_48, D_49, D_5, D_50, D_51, D_52, D_53, D_54, D_55, D_56, D_57, D_58, D_59, D_6, D_60, D_61, D_62, D_63, D_64, D_65, D_66, D_67, D_68, D_69, D_7, D_70, D_71, D_72, D_73, D_74, D_75, D_8, D_9: Diode SOD-323, Diode_SMD:D_SOD-323_HandSoldering, symbol Device:D_Small
- removed K_0, K_1, K_10, K_11, K_12, K_14, K_15, K_17, K_18, K_19, K_2, K_20, K_21, K_22, K_23, K_24, K_25, K_26, K_27, K_28, K_3, K_30, K_31, K_33, K_34, K_35, K_36, K_37, K_38, K_39, K_4, K_40, K_41, K_42, K_43, K_44, K_45, K_46, K_48, K_49, K_5, K_50, K_51, K_52, K_53, K_54, K_55, K_56, K_57, K_58, K_6, K_60, K_61, K_62, K_69, K_7, K_70, K_71, K_72, K_73, K_74, K_75, K_8, K_9: KEYSW, MX_Only:MXOnly-1U-NoLED, symbol MX_Alps_Hybrid:MX-NoLED
- removed K_13: KEYSW, MX_Only:MXOnly-2U-NoLED, symbol MX_Alps_Hybrid:MX-NoLED
- removed K_16: KEYSW, MX_Only:MXOnly-1.5U-NoLED, symbol MX_Alps_Hybrid:MX-NoLED
- removed K_29: KEYSW, MX_Only:MXOnly-ISO-ROTATED-ReversedStabilizers-NoLED, symbol MX_Alps_Hybrid:MX-NoLED
- removed K_32, K_59, K_67: KEYSW, MX_Only:MXOnly-1.75U-NoLED, symbol MX_Alps_Hybrid:MX-NoLED
- removed K_47, K_63, K_64, K_65: KEYSW, MX_Only:MXOnly-1.25U-NoLED, symbol MX_Alps_Hybrid:MX-NoLED
- removed K_66, K_68: KEYSW, MX_Only:MXOnly-2.25U-ReversedStabilizers-NoLED, symbol MX_Alps_Hybrid:MX-NoLED
- removed U1: Pico, MCU_RaspberryPi_and_Boards:RPi_Pico_SMD_TH, symbol MCU_RaspberryPi_and_Boards:Pico
Connections:
- net labels removed: col0, col1, col10, col11, col12, col13, col14, col15, col16, col2, col3, col4, col5, col6, col7, col8, col9, gnd, row0, row1, row2, row3, row4
- wire segments 304 -> 0
