File: TopPCB/EnvKB65-SwitchPlate.sch (KiCad schematic (older format))
At the start: 6 parts

Commit message: See List
* removed RP2040 and atmega32u4 versions
* updated main PCB to have larger holes
* fixed some stuff on the main PCB and added some labels
Parts:
- H1, H2, H3, H4, H5, H6: symbol Mechanical:MountingHole -> Mechanical:MountingHole_Pad
Connections:
- new net GND: H1.1, H2.1, H3.1, H4.1, H5.1, H6.1
Changed lines of the file:
@@
 $EndDescr
 $Comp
-L Mechanical:MountingHole H1
+L Mechanical:MountingHole_Pad H3
+U 1 1 60AE412B
+P 5450 6150
+F 0 "H3" H 5550 6196 50  0000 L CNN
+F 1 "MountingHole" H 5550 6105 50  0001 L CNN
+F 2 "MountingHole:MountingHole_2.2mm_M2_Pad" H 5450 6150 50  0001 C CNN
+F 3 "~" H 5450 6150 50  0001 C CNN
+	1    5450 6150
+	1    0    0    -1
+$EndComp
+$Comp
+L Mechanical:MountingHole_Pad H4
+U 1 1 60AFC1C3
+P 5750 6150
+F 0 "H4" H 5850 6196 50  0000 L CNN
+F 1 "MountingHole" H 5850 6105 50  0001 L CNN
+F 2 "MountingHole:MountingHole_2.2mm_M2_Pad" H 5750 6150 50  0001 C CNN
+F 3 "~" H 5750 6150 50  0001 C CNN
+	1    5750 6150
+	1    0    0    -1
+$EndComp
+$Comp
+L Mechanical:MountingHole_Pad H5
+U 1 1 60B142B5
+P 6050 6150
+F 0 "H5" H 6150 6196 50  0000 L CNN
+F 1 "MountingHole" H 6150 6105 50  0001 L CNN
+F 2 "MountingHole:MountingHole_2.2mm_M2_Pad" H 6050 6150 50  0001 C CNN
+F 3 "~" H 6050 6150 50  0001 C CNN
+	1    6050 6150
+	1    0    0    -1
+$EndComp
+$Comp
+L Mechanical:MountingHole_Pad H6
+U 1 1 60B2C4B8
+P 6350 6150
+F 0 "H6" H 6450 6196 50  0000 L CNN
+F 1 "MountingHole" H 6450 6105 50  0001 L CNN
+F 2 "MountingHole:MountingHole_2.2mm_M2_Pad" H 6350 6150 50  0001 C CNN
+F 3 "~" H 6350 6150 50  0001 C CNN
+	1    6350 6150
+	1    0    0    -1
+$EndComp
+$Comp
+L Mechanical:MountingHole_Pad H1
 U 1 1 60AC66FB
 P 4850 6150
 F 0 "H1" H 4950 6196 50  0000 L CNN
-F 1 "MountingHole" H 4950 6105 50  0000 L CNN
+F 1 "MountingHole" H 4950 6105 50  0001 L CNN
 F 2 "MountingHole:MountingHole_2.2mm_M2_Pad" H 4850 6150 50  0001 C CNN
 F 3 "~" H 4850 6150 50  0001 C CNN
@@
 $EndComp
 $Comp
-L Mechanical:MountingHole H2
+L Mechanical:MountingHole_Pad H2
 U 1 1 60ACBE92
-P 4850 6350
-F 0 "H2" H 4950 6396 50  0000 L CNN
-F 1 "MountingHole" H 4950 6305 50  0000 L CNN
-F 2 "MountingHole:MountingHole_2.2mm_M2_Pad" H 4850 6350 50  0001 C CNN
-F 3 "~" H 4850 6350 50  0001 C CNN
-	1    4850 6350
+P 5150 6150
+F 0 "H2" H 5250 6196 50  0000 L CNN
+F 1 "MountingHole" H 5250 6105 50  0001 L CNN
+F 2 "MountingHole:MountingHole_2.2mm_M2_Pad" H 5150 6150 50  0001 C CNN
+F 3 "~" H 5150 6150 50  0001 C CNN
+	1    5150 6150
 	1    0    0    -1
 $EndComp
+Wire Wire Line
+	4850 6250 5150 6250
+Wire Wire Line
+	6350 6250 6350 6300
+Connection ~ 6350 6250
+Connection ~ 5150 6250
+Wire Wire Line
+	5150 6250 5450 6250
+Connection ~ 5450 6250
+Wire Wire Line
+	5450 6250 5750 6250
+Connection ~ 5750 6250
+Wire Wire Line
+	5750 6250 6050 6250
+Connection ~ 6050 6250
+Wire Wire Line
+	6050 6250 6350 6250
 $Comp
-L Mechanical:MountingHole H3
-U 1 1 60AE412B
-P 4850 6550
-F 0 "H3" H 4950 6596 50  0000 L CNN
-F 1 "MountingHole" H 4950 6505 50  0000 L CNN
-F 2 "MountingHole:MountingHole_2.2mm_M2_Pad" H 4850 6550 50  0001 C CNN
-F 3 "~" H 4850 6550 50  0001 C CNN
-	1    4850 6550
+L power:GND #PWR?
+U 1 1 615E0DF6
+P 6350 6300
+F 0 "#PWR?" H 6350 6050 50  0001 C CNN
+F 1 "GND" H 6355 6127 50  0000 C CNN
+F 2 "" H 6350 6300 50  0001 C CNN
+F 3 "" H 6350 6300 50  0001 C CNN
+	1    6350 6300
 	1    0    0    -1
 $EndComp
-$Comp
-L Mechanical:MountingHole H4
-U 1 1 60AFC1C3
-P 4850 6750
-F 0 "H4" H 4950 6796 50  0000 L CNN
-F 1 "MountingHole" H 4950 6705 50  0000 L CNN
-F 2 "MountingHole:MountingHole_2.2mm_M2_Pad" H 4850 6750 50  0001 C CNN
-F 3 "~" H 4850 6750 50  0001 C CNN
-	1    4850 6750
-	1    0    0    -1
-$EndComp
-$Comp
-L Mechanical:MountingHole H5
-U 1 1 60B142B5
-P 4850 6950
-F 0 "H5" H 4950 6996 50  0000 L CNN
-F 1 "MountingHole" H 4950 6905 50  0000 L CNN
-F 2 "MountingHole:MountingHole_2.2mm_M2_Pad" H 4850 6950 50  0001 C CNN
-F 3 "~" H 4850 6950 50  0001 C CNN
-	1    4850 6950
-	1    0    0    -1
-$EndComp
-$Comp
-L Mechanical:MountingHole H6
-U 1 1 60B2C4B8
-P 4850 7150
-F 0 "H6" H 4950 7196 50  0000 L CNN
-F 1 "MountingHole" H 4950 7105 50  0000 L CNN
-F 2 "MountingHole:MountingHole_2.2mm_M2_Pad" H 4850 7150 50  0001 C CNN
-F 3 "~" H 4850 7150 50  0001 C CNN
-	1    4850 7150
-	1    0    0    -1
-$EndComp
