File: TopPCB/EnvKB65-SwitchPlate.kicad_pcb (KiCad board)
At the start: 2 copper layers, 326.8 x 101 mm, 5 parts

Commit message: Generated some Gerbers and added some testing graphics for now.
Parts:
- removed the H6 at (251.1, 182.0)
- added G***: LOGO, Logo:patern, F.Cu at (225.2, 148.1)
- added H2: MountingHole, MountingHole:MountingHole_2.2mm_M2_Pad, F.Cu at (69.0, 101.0)
- added H3: MountingHole, MountingHole:MountingHole_2.2mm_M2_Pad, F.Cu at (86.8, 185.2)
- added H4: MountingHole, MountingHole:MountingHole_2.2mm_M2_Pad, F.Cu at (367.8, 178.2)
- added H5: MountingHole, MountingHole:MountingHole_2.2mm_M2_Pad, F.Cu at (224.9, 121.6)
- added H6 (x2): MountingHole, MountingHole:MountingHole_2.2mm_M2_Pad, F.Cu at (251.1, 183.5)

Commit message: See List
* removed RP2040 and atmega32u4 versions
* updated main PCB to have larger holes
* fixed some stuff on the main PCB and added some labels
Connections:
- H2 pad 1: (no net) -> GND (x2)
- H3 pad 1: (no net) -> GND (x2)
- H4 pad 1: (no net) -> GND (x2)
- H5 pad 1: (no net) -> GND (x2)
- H6 pad 1: (no net) -> GND (x2)
Routing:
- added copper zone on B.Cu, net GND
- added copper zone on F.Cu, net GND
- removed copper zone on B.Cu, net (none)
- removed copper zone on F.Cu, net (none)
Other:
- board text added: "Mechboards.co.uk"

Commit message: some small fixes
Other:
- net class Default removed
