File: TopPCB/EnvKB65-SwitchPlate.kicad_pcb (KiCad board)
At the start: 2 copper layers, 326.8 x 101 mm, 11 parts

Commit message: Removed Mechboards branding as there is now a mechboards fork
Parts:
- removed G***: LOGO, Logo:patern
- added kibuzzard-629271A1: G***, kibuzzard-629271A1, F.Cu at (333.8, 101.2)
Other:
- board text removed: "Mechboards.co.uk"
