File: BottomPCB/EnvKB65_bottom.sch (KiCad schematic (older format))
At the start: 7 parts, among them J1 Conn_01x01_Female

Commit message: Mount hole tweak to allow for switches to seat properly with a spacer installed
Parts:
- removed J1: Conn_01x01_Female, TestPoint:TestPoint_Pad_1.0x1.0mm, symbol Connector:Conn_01x01_Female
Changed lines of the file:
@@
 	1    0    0    -1
 $EndComp
-$Comp
-L Connector:Conn_01x01_Female J1
-U 1 1 60A43BB1
-P 4000 6450
-F 0 "J1" H 4028 6476 50  0000 L CNN
-F 1 "Conn_01x01_Female" H 4028 6385 50  0000 L CNN
-F 2 "TestPoint:TestPoint_Pad_1.0x1.0mm" H 4000 6450 50  0001 C CNN
-F 3 "~" H 4000 6450 50  0001 C CNN
-	1    4000 6450
-	1    0    0    -1
-$EndComp
-Text GLabel 3800 6450 0    50   Input ~ 0
-GND
 $EndSCHEMATC

Commit message: replaced all mount holes with versions that have pads
I did this because the pcb can get scraped up if you take it apart a bunch of times to clean it, hopefully this mitigates that.
Parts:
- H1, H2, H3, H4, H5, H6: footprint MountingHole:MountingHole_2.2mm_M2 -> MountingHole:MountingHole_2.2mm_M2_Pad
Changed lines of the file:
@@
 F 0 "H1" H 4950 6196 50  0000 L CNN
 F 1 "MountingHole" H 4950 6105 50  0000 L CNN
-F 2 "MountingHole:MountingHole_2.2mm_M2" H 4850 6150 50  0001 C CNN
+F 2 "MountingHole:MountingHole_2.2mm_M2_Pad" H 4850 6150 50  0001 C CNN
 F 3 "~" H 4850 6150 50  0001 C CNN
 	1    4850 6150
@@
 F 0 "H2" H 4950 6396 50  0000 L CNN
 F 1 "MountingHole" H 4950 6305 50  0000 L CNN
-F 2 "MountingHole:MountingHole_2.2mm_M2" H 4850 6350 50  0001 C CNN
+F 2 "MountingHole:MountingHole_2.2mm_M2_Pad" H 4850 6350 50  0001 C CNN
 F 3 "~" H 4850 6350 50  0001 C CNN
 	1    4850 6350
@@
 F 0 "H3" H 4950 6596 50  0000 L CNN
 F 1 "MountingHole" H 4950 6505 50  0000 L CNN
-F 2 "MountingHole:MountingHole_2.2mm_M2" H 4850 6550 50  0001 C CNN
+F 2 "MountingHole:MountingHole_2.2mm_M2_Pad" H 4850 6550 50  0001 C CNN
 F 3 "~" H 4850 6550 50  0001 C CNN
 	1    4850 6550
@@
 F 0 "H4" H 4950 6796 50  0000 L CNN
 F 1 "MountingHole" H 4950 6705 50  0000 L CNN
-F 2 "MountingHole:MountingHole_2.2mm_M2" H 4850 6750 50  0001 C CNN
+F 2 "MountingHole:MountingHole_2.2mm_M2_Pad" H 4850 6750 50  0001 C CNN
 F 3 "~" H 4850 6750 50  0001 C CNN
 	1    4850 6750
@@
 F 0 "H5" H 4950 6996 50  0000 L CNN
 F 1 "MountingHole" H 4950 6905 50  0000 L CNN
-F 2 "MountingHole:MountingHole_2.2mm_M2" H 4850 6950 50  0001 C CNN
+F 2 "MountingHole:MountingHole_2.2mm_M2_Pad" H 4850 6950 50  0001 C CNN
 F 3 "~" H 4850 6950 50  0001 C CNN
 	1    4850 6950
@@
 F 0 "H6" H 4950 7196 50  0000 L CNN
 F 1 "MountingHole" H 4950 7105 50  0000 L CNN
-F 2 "MountingHole:MountingHole_2.2mm_M2" H 4850 7150 50  0001 C CNN
+F 2 "MountingHole:MountingHole_2.2mm_M2_Pad" H 4850 7150 50  0001 C CNN
 F 3 "~" H 4850 7150 50  0001 C CNN
 	1    4850 7150
