File: MainPCB-HOTSWAP/EnvKB65.kicad_pcb (KiCad board)
At the start: 2 copper layers, 320.8 x 99.3 mm, 157 parts, among them U0 Pico

Commit message: small cleanup + worked on routing races and all
Parts:
- moved D_40 4.57 mm to (325.7, 160.8), turned to 270 degrees
- moved D_42 3.97 mm to (88.6, 178.1), turned to 180 degrees
- turned K_27 to 270 degrees
- turned K_28 to 180 degrees
- turned K_42 to 90 degrees
- turned K_43 to 180 degrees
- turned ST6 to 90 degrees
Routing:
- net row1: track 324.2 -> 298.4 mm
- net Net-(D_40-Pad2): track 14.8 -> 26.4 mm, vias 0 -> 1
- net col0: track 389.0 -> 400.0 mm
- net Net-(D_27-Pad2): track 24.9 -> 15.0 mm
- net col14: track 140.1 -> 131.7 mm
- net row3: track 350.3 -> 343.0 mm, vias 0 -> 1
- net Net-(D_41-Pad2): track 31.4 -> 35.8 mm
- net Net-(D_57-Pad2): track 17.7 -> 20.5 mm
- net row4: track 348.7 -> 351.1 mm, vias 0 -> 4
- net Net-(D_70-Pad2): track 16.7 -> 18.6 mm
- net col7: track 236.5 -> 238.3 mm
- net col5: track 272.5 -> 274.1 mm
- net row2: track 314.4 -> 315.9 mm
- net col10: track 206.6 -> 208.1 mm
- net col6: track 275.2 -> 276.5 mm
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Other:
- board text added: "http://github.com/Envious-Data/Env-KB65MHS"
- board text removed: "http://github.com/Envious-Data/Env-KB65M"

Commit message: fixed some trace and pad/hole conflictions and spaced some traces although not causing DRC errors.
Routing:
- net Net-(D_27-Pad2): track 15.0 -> 42.9 mm, vias 0 -> 1
- net row1: track 298.4 -> 318.4 mm, vias 0 -> 2
- net Net-(D_41-Pad2): track 35.8 -> 51.1 mm, vias 0 -> 2
- net col14: track 131.7 -> 137.6 mm
- net row0: track 354.1 -> 356.4 mm
- net row4: track 351.1 -> 349.2 mm
- net col7: track 238.3 -> 236.5 mm
- net col2: track 326.6 -> 325.3 mm
- net col8: track 238.8 -> 237.6 mm
- net col3: track 333.4 -> 332.2 mm
- net col1: track 355.6 -> 354.6 mm
- net col0: track 400.0 -> 399.0 mm
- net col12: track 174.9 -> 174.1 mm
- net (no net): track 0.73 -> 0.00 mm
- net col10: track 208.1 -> 207.4 mm
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Other:
- rule trace_min: 0.2 -> 0.127
