File: MainPCB-HOTSWAP/EnvKB65HS.kicad_pcb (KiCad board)
At the start: 2 copper layers, 320.8 x 99.3 mm, 157 parts, among them U0 Pico

Commit message: corrected hotswap socket being cut off on the left side (PCB is slightly wider)
Other:
- board size 320.8 x 99.3 mm -> 322.3 x 99.3 mm

Commit message: adjusted design and fixed issues, Generated updated gerber
Parts:
- H0, H1, H2, H3, H4, H5: footprint MountingHole:MountingHole_4.3mm_M4 -> MountingHole:MountingHole_2.2mm_M2_Pad_Via
Connections:
- H0 pad 1: (no net) -> GND
- H1 pad 1: (no net) -> GND
- H2 pad 1: (no net) -> GND
- H3 pad 1: (no net) -> GND
- H4 pad 1: (no net) -> GND
- H5 pad 1: (no net) -> GND
- U0 pad 13: gnd -> GND
- U0 pad 18: gnd -> GND
- U0 pad 23: gnd -> GND
- U0 pad 28: gnd -> GND
- U0 pad 3: gnd -> GND
- U0 pad 33: gnd -> GND
- U0 pad 38: gnd -> GND
- U0 pad 8: gnd -> GND
Routing:
- net col11: track 189.1 -> 187.0 mm
- net col9: track 201.5 -> 199.8 mm
- net col4: track 310.5 -> 309.0 mm
- net col12: track 174.1 -> 175.2 mm
- net col5: track 274.1 -> 273.2 mm
- net col10: track 207.4 -> 206.6 mm
- net row3: track 342.5 -> 343.2 mm
- net col6: track 276.5 -> 275.8 mm
- net col1: track 354.6 -> 354.1 mm
- net gnd: vias 6 -> 0
- net GND: vias 0 -> 5
- added copper zone on B.Cu, net GND
- added copper zone on F.Cu, net GND
- removed copper zone on B.Cu, net gnd
- removed copper zone on F.Cu, net gnd
Other:
- net class Default: clearance 0.4 -> 0.127
- rule trace_clearance: 0.4 -> 0.127
