File: MainPCB-HOTSWAP/EnvKB65HS.kicad_pcb (KiCad board)
At the start: 2 copper layers, 322.3 x 99.3 mm, 160 parts, among them J1 Conn_01x04, U0 Pico

Commit message: larger holes for aliexpress smd mounts
Parts:
- moved kibuzzard-62927A63 1.94 mm to (90.3, 100.7)
Routing:
- net col0: track 393.5 -> 392.1 mm
Changed lines of the file:
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@@
       (psa4output false)
       (plotreference true)
-      (plotvalue false)
-      (plotinvisibletext false)
+      (plotvalue true)
+      (plotinvisibletext true)
       (sketchpadsonfab false)
       (subtractmaskfromsilk true)
@@
     (pad "37" thru_hole oval locked (at 8.89 -16.51) (size 1.7 1.7) (drill 1.02) (layers *.Cu *.Mask)
       (net 101 "unconnected-(U0-Pad37)") (pinfunction "3V3_EN") (pintype "input"))
-    (pad "38" smd rect locked (at 8.89 -19.05) (size 3.5 1.7) (drill (offset 0.9 0)) (layers "F.Cu" "F.Mask")
+    (pad "38" smd rect locked (at 8.89 -19.05) (size 1.7 1.7) (layers "F.Cu" "F.Mask")
       (net 104 "GND") (pinfunction "GND") (pintype "bidirectional"))
     (pad "38" thru_hole rect locked (at 8.89 -19.05) (size 1.7 1.7) (drill 1.02) (layers *.Cu *.Mask)
@@
     (property "Sheetname" "")
     (attr exclude_from_pos_files)
-    (fp_text reference "H1" (at 0 -3.2) (layer "F.SilkS")
+    (fp_text reference "H1" (at 0 -3.2) (layer "F.Fab")
       (effects (font (size 1 1) (thickness 0.15)))
     )
@@
     (fp_circle (center 0 0) (end 2.2 0) (layer "Cmts.User") (width 0.15) (fill none))
     (fp_circle (center 0 0) (end 2.45 0) (layer "F.CrtYd") (width 0.05) (fill none))
-    (pad "1" thru_hole circle (at 0 0) (size 5.3 5.3) (drill 3) (layers *.Cu *.Mask)
+    (pad "1" thru_hole circle (at 0 0) (size 6 6) (drill 3.8) (layers *.Cu *.Mask)
       (net 106 "unconnected-(H1-Pad1)") (pinfunction "1") (pintype "input+no_connect"))
   )
@@
     (property "Sheetname" "")
     (attr exclude_from_pos_files)
-    (fp_text reference "H2" (at 0 -3.2) (layer "F.SilkS")
+    (fp_text reference "H2" (at 0 -3.2) (layer "F.Fab")
       (effects (font (size 1 1) (thickness 0.15)))
     )
@@
     (fp_circle (center 0 0) (end 2.2 0) (layer "Cmts.User") (width 0.15) (fill none))
     (fp_circle (center 0 0) (end 2.45 0) (layer "F.CrtYd") (width 0.05) (fill none))
-    (pad "1" thru_hole circle (at 0 0) (size 5.3 5.3) (drill 3) (layers *.Cu *.Mask)
+    (pad "1" thru_hole circle (at 0 0) (size 6 6) (drill 3.8) (layers *.Cu *.Mask)
       (net 107 "unconnected-(H2-Pad1)") (pinfunction "1") (pintype "input+no_connect"))
   )
@@
     (property "Sheetname" "")
     (attr exclude_from_pos_files)
-    (fp_text reference "H3" (at 0 -3.2) (layer "F.SilkS")
+    (fp_text reference "H3" (at 0 -3.2) (layer "F.Fab")
       (effects (font (size 1 1) (thickness 0.15)))
     )
@@
     (fp_circle (center 0 0) (end 2.2 0) (layer "Cmts.User") (width 0.15) (fill none))
     (fp_circle (center 0 0) (end 2.45 0) (layer "F.CrtYd") (width 0.05) (fill none))
-    (pad "1" thru_hole circle (at 0 0) (size 5.3 5.3) (drill 3) (layers *.Cu *.Mask)
+    (pad "1" thru_hole circle (at 0 0) (size 6 6) (drill 3.8) (layers *.Cu *.Mask)
       (net 108 "unconnected-(H3-Pad1)") (pinfunction "1") (pintype "input+no_connect"))
   )
@@
     (property "Sheetname" "")
     (attr exclude_from_pos_files)
-    (fp_text reference "H4" (at 0 -3.2) (layer "F.SilkS")
+    (fp_text reference "H4" (at 0 -3.2) (layer "F.Fab")
       (effects (font (size 1 1) (thickness 0.15)))
     )
@@
     (fp_circle (center 0 0) (end 2.2 0) (layer "Cmts.User") (width 0.15) (fill none))
     (fp_circle (center 0 0) (end 2.45 0) (layer "F.CrtYd") (width 0.05) (fill none))
-    (pad "1" thru_hole circle (at 0 0) (size 5.3 5.3) (drill 3) (layers *.Cu *.Mask)
+    (pad "1" thru_hole circle (at 0 0) (size 6 6) (drill 3.8) (layers *.Cu *.Mask)
       (net 109 "unconnected-(H4-Pad1)") (pinfunction "1") (pintype "input+no_connect"))
   )
@@
     (property "Sheetname" "")
     (attr exclude_from_pos_files)
-    (fp_text reference "H0" (at 0 -3.2) (layer "F.SilkS")
+    (fp_text reference "H0" (at 0 -3.2) (layer "F.Fab")
       (effects (font (size 1 1) (thickness 0.15)))
     )
@@
     (fp_circle (center 0 0) (end 2.2 0) (layer "Cmts.User") (width 0.15) (fill none))
     (fp_circle (center 0 0) (end 2.45 0) (layer "F.CrtYd") (width 0.05) (fill none))
-    (pad "1" thru_hole circle (at 0 0) (size 5.3 5.3) (drill 3) (layers *.Cu *.Mask)
+    (pad "1" thru_hole circle (at 0 0) (size 6 6) (drill 3.8) (layers *.Cu *.Mask)
       (net 105 "unconnected-(H0-Pad1)") (pinfunction "1") (pintype "input+no_connect"))
   )
@@
     (property "Sheetname" "")
     (attr exclude_from_pos_files)
-    (fp_text reference "H5" (at 0 -3.2) (layer "F.SilkS")
+    (fp_text reference "H5" (at 0 -3.2) (layer "F.Fab")
       (effects (font (size 1 1) (thickness 0.15)))
     )
@@
     (fp_circle (center 0 0) (end 2.2 0) (layer "Cmts.User") (width 0.15) (fill none))
     (fp_circle (center 0 0) (end 2.45 0) (layer "F.CrtYd") (width 0.05) (fill none))
-    (pad "1" thru_hole circle (at 0 0) (size 5.3 5.3) (drill 3) (layers *.Cu *.Mask)
+    (pad "1" thru_hole circle (at 0 0) (size 6 6) (drill 3.8) (layers *.Cu *.Mask)
       (net 110 "unconnected-(H5-Pad1)") (pinfunction "1") (pintype "input+no_connect"))
   )
@@
     (property "Sheetname" "")
     (attr exclude_from_pos_files)
-    (fp_text reference "ST7" (at 0 -3) (layer "F.SilkS")
+    (fp_text reference "ST7" (at 0 -3) (layer "F.Fab")
       (effects (font (size 1 1) (thickness 0.15)))
     )
@@
   )
   (footprint "kibuzzard-62927A63" (layer "F.Cu")
-    (at 88.4 100.7)
+    (at 90.339654 100.7)
     (descr "Converted using: scripting")
     (tags "svg2mod")
     (attr board_only exclude_from_pos_files exclude_from_bom)
-    (fp_text reference "kibuzzard-62927A63" (at 0 -2.376996) (layer "F.SilkS") hide
+    (fp_text reference "kibuzzard-62927A63" (at 0 -2.376996) (layer "F.Fab") hide
       (effects (font (size 0.000254 0.000254) (thickness 0.000003)))
     )
@@
     (property "Sheetname" "")
     (attr through_hole)
-    (fp_text reference "J1" (at 0 -2.77 90) (layer "F.SilkS")
+    (fp_text reference "J1" (at 0 -2.77 90) (layer "F.Fab")
       (effects (font (size 1 1) (thickness 0.15)))
     )
@@
   (arc (start 82.454416 177.9) (mid 84.806229 177.432195) (end 86.8 176.1) (width 0.25) (layer "F.Cu") (net 1))
   (arc (start 76.3 177.600058) (mid 75.929691 175.738387) (end 74.875138 174.160138) (width 0.25) (layer "F.Cu") (net 1))
-  (segment (start 356.65369 100.33) (end 77.338301 100.33) (width 0.25) (layer "B.Cu") (net 1))
+  (segment (start 356.65369 100.33) (end 79.93 100.33) (width 0.25) (layer "B.Cu") (net 1))
   (segment (start 358.89 99.02) (end 358.235 99.675) (width 0.25) (layer "B.Cu") (net 1))
-  (arc (start 77.338301 100.33) (mid 71.229527 102.860341) (end 68.6992 108.96912) (width 0.25) (layer "B.Cu") (net 1))
+  (segment (start 68.6992 108.96912) (end 75.505725 102.162595) (width 0.25) (layer "B.Cu") (net 1))
   (arc (start 358.235 99.675) (mid 357.509488 100.159771) (end 356.65369 100.33) (width 0.25) (layer "B.Cu") (net 1))
+  (arc (start 75.505725 102.162595) (mid 77.535599 100.806276) (end 79.93 100.33) (width 0.25) (layer "B.Cu") (net 1))
   (segment (start 92.5117 166.11912) (end 92.5117 161.325302) (width 0.25) (layer "F.Cu") (net 2))
   (segment (start 93.1 180.840556) (end 93.1 166.70742) (width 0.25) (layer "F.Cu") (net 2))

Commit message: swapped mount holes back and generated updated gerbers and etc
Parts:
- H0, H1, H2, H3, H4, H5: value SMTWE2020MTJ -> C2928180; footprint Logo:MountingHole_3mm_Pad5.3mm -> MountingHole:MountingHole_3.5mm
Changed lines of the file:
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@@
   (net 103 "GPIO28")
   (net 104 "GND")
-  (net 105 "unconnected-(H0-Pad1)")
-  (net 106 "unconnected-(H1-Pad1)")
-  (net 107 "unconnected-(H2-Pad1)")
-  (net 108 "unconnected-(H3-Pad1)")
-  (net 109 "unconnected-(H4-Pad1)")
-  (net 110 "unconnected-(H5-Pad1)")
   (footprint "MX_Only:MXOnly-1U-Hotswap-Modified" (layer "F.Cu")
     (at 196.3342 130.55912)
@@
       (net 36 "Net-(D_13-Pad2)") (pinfunction "ROW") (pintype "passive"))
   )
-  (footprint "Logo:MountingHole_3mm_Pad5.3mm" (layer "F.Cu")
+  (footprint "MountingHole:MountingHole_3.5mm" (layer "F.Cu")
     (at 69 101)
-    (descr "Mounting Hole 2.2mm, M2")
-    (tags "mounting hole 2.2mm m2")
+    (descr "Mounting Hole 3.5mm, no annular")
+    (tags "mounting hole 3.5mm no annular")
     (property "Sheetfile" "EnvKB65HS.kicad_sch")
     (property "Sheetname" "")
     (attr exclude_from_pos_files)
-    (fp_text reference "H1" (at 0 -3.2) (layer "F.Fab")
-      (effects (font (size 1 1) (thickness 0.15)))
-    )
-    (fp_text value "SMTWE2020MTJ" (at 0 3.2) (layer "F.Fab")
+    (fp_text reference "H1" (at 0 -4.5) (layer "F.SilkS")
+      (effects (font (size 1 1) (thickness 0.15)))
+    )
+    (fp_text value "C2928180" (at 0 4.5) (layer "F.Fab")
       (effects (font (size 1 1) (thickness 0.15)))
     )
@@
       (effects (font (size 1 1) (thickness 0.15)))
     )
-    (fp_circle (center 0 0) (end 2.2 0) (layer "Cmts.User") (width 0.15) (fill none))
-    (fp_circle (center 0 0) (end 2.45 0) (layer "F.CrtYd") (width 0.05) (fill none))
-    (pad "1" thru_hole circle (at 0 0) (size 6 6) (drill 3.8) (layers *.Cu *.Mask)
-      (net 106 "unconnected-(H1-Pad1)") (pinfunction "1") (pintype "input+no_connect"))
-  )
-  (footprint "Logo:MountingHole_3mm_Pad5.3mm" (layer "F.Cu")
+    (fp_circle (center 0 0) (end 3.5 0) (layer "Cmts.User") (width 0.15) (fill none))
+    (fp_circle (center 0 0) (end 3.75 0) (layer "F.CrtYd") (width 0.05) (fill none))
+    (pad "" np_thru_hole circle (at 0 0) (size 3.5 3.5) (drill 3.5) (layers *.Cu *.Mask))
+  )
+  (footprint "MountingHole:MountingHole_3.5mm" (layer "F.Cu")
     (at 86.8 185.22)
-    (descr "Mounting Hole 2.2mm, M2")
-    (tags "mounting hole 2.2mm m2")
+    (descr "Mounting Hole 3.5mm, no annular")
+    (tags "mounting hole 3.5mm no annular")
     (property "Sheetfile" "EnvKB65HS.kicad_sch")
     (property "Sheetname" "")
     (attr exclude_from_pos_files)
-    (fp_text reference "H2" (at 0 -3.2) (layer "F.Fab")
-      (effects (font (size 1 1) (thickness 0.15)))
-    )
-    (fp_text value "SMTWE2020MTJ" (at 0 3.2) (layer "F.Fab")
+    (fp_text reference "H2" (at 0 -4.5) (layer "F.SilkS")
+      (effects (font (size 1 1) (thickness 0.15)))
+    )
+    (fp_text value "C2928180" (at 0 4.5) (layer "F.Fab")
       (effects (font (size 1 1) (thickness 0.15)))
     )
@@
       (effects (font (size 1 1) (thickness 0.15)))
     )
-    (fp_circle (center 0 0) (end 2.2 0) (layer "Cmts.User") (width 0.15) (fill none))
-    (fp_circle (center 0 0) (end 2.45 0) (layer "F.CrtYd") (width 0.05) (fill none))
-    (pad "1" thru_hole circle (at 0 0) (size 6 6) (drill 3.8) (layers *.Cu *.Mask)
-      (net 107 "unconnected-(H2-Pad1)") (pinfunction "1") (pintype "input+no_connect"))
-  )
-  (footprint "Logo:MountingHole_3mm_Pad5.3mm" (layer "F.Cu")
+    (fp_circle (center 0 0) (end 3.5 0) (layer "Cmts.User") (width 0.15) (fill none))
+    (fp_circle (center 0 0) (end 3.75 0) (layer "F.CrtYd") (width 0.05) (fill none))
+    (pad "" np_thru_hole circle (at 0 0) (size 3.5 3.5) (drill 3.5) (layers *.Cu *.Mask))
+  )
+  (footprint "MountingHole:MountingHole_3.5mm" (layer "F.Cu")
     (at 367.8 178.2)
-    (descr "Mounting Hole 2.2mm, M2")
-    (tags "mounting hole 2.2mm m2")
+    (descr "Mounting Hole 3.5mm, no annular")
+    (tags "mounting hole 3.5mm no annular")
     (property "Sheetfile" "EnvKB65HS.kicad_sch")
     (property "Sheetname" "")
     (attr exclude_from_pos_files)
-    (fp_text reference "H3" (at 0 -3.2) (layer "F.Fab")
-      (effects (font (size 1 1) (thickness 0.15)))
-    )
-    (fp_text value "SMTWE2020MTJ" (at 0 3.2) (layer "F.Fab")
+    (fp_text reference "H3" (at 0 -4.5) (layer "F.SilkS")
+      (effects (font (size 1 1) (thickness 0.15)))
+    )
+    (fp_text value "C2928180" (at 0 4.5) (layer "F.Fab")
       (effects (font (size 1 1) (thickness 0.15)))
     )
@@
       (effects (font (size 1 1) (thickness 0.15)))
     )
-    (fp_circle (center 0 0) (end 2.2 0) (layer "Cmts.User") (width 0.15) (fill none))
-    (fp_circle (center 0 0) (end 2.45 0) (layer "F.CrtYd") (width 0.05) (fill none))
-    (pad "1" thru_hole circle (at 0 0) (size 6 6) (drill 3.8) (layers *.Cu *.Mask)
-      (net 108 "unconnected-(H3-Pad1)") (pinfunction "1") (pintype "input+no_connect"))
-  )
-  (footprint "Logo:MountingHole_3mm_Pad5.3mm" (layer "F.Cu")
+    (fp_circle (center 0 0) (end 3.5 0) (layer "Cmts.User") (width 0.15) (fill none))
+    (fp_circle (center 0 0) (end 3.75 0) (layer "F.CrtYd") (width 0.05) (fill none))
+    (pad "" np_thru_hole circle (at 0 0) (size 3.5 3.5) (drill 3.5) (layers *.Cu *.Mask))
+  )
+  (footprint "MountingHole:MountingHole_3.5mm" (layer "F.Cu")
     (at 224.9 121.6)
-    (descr "Mounting Hole 2.2mm, M2")
-    (tags "mounting hole 2.2mm m2")
+    (descr "Mounting Hole 3.5mm, no annular")
+    (tags "mounting hole 3.5mm no annular")
     (property "Sheetfile" "EnvKB65HS.kicad_sch")
     (property "Sheetname" "")
     (attr exclude_from_pos_files)
-    (fp_text reference "H4" (at 0 -3.2) (layer "F.Fab")
-      (effects (font (size 1 1) (thickness 0.15)))
-    )
-    (fp_text value "SMTWE2020MTJ" (at 0 3.2) (layer "F.Fab")
+    (fp_text reference "H4" (at 0 -4.5) (layer "F.SilkS")
+      (effects (font (size 1 1) (thickness 0.15)))
+    )
+    (fp_text value "C2928180" (at 0 4.5) (layer "F.Fab")
       (effects (font (size 1 1) (thickness 0.15)))
     )
@@
       (effects (font (size 1 1) (thickness 0.15)))
     )
-    (fp_circle (center 0 0) (end 2.2 0) (layer "Cmts.User") (width 0.15) (fill none))
-    (fp_circle (center 0 0) (end 2.45 0) (layer "F.CrtYd") (width 0.05) (fill none))
-    (pad "1" thru_hole circle (at 0 0) (size 6 6) (drill 3.8) (layers *.Cu *.Mask)
-      (net 109 "unconnected-(H4-Pad1)") (pinfunction "1") (pintype "input+no_connect"))
-  )
-  (footprint "Logo:MountingHole_3mm_Pad5.3mm" (layer "F.Cu")
+    (fp_circle (center 0 0) (end 3.5 0) (layer "Cmts.User") (width 0.15) (fill none))
+    (fp_circle (center 0 0) (end 3.75 0) (layer "F.CrtYd") (width 0.05) (fill none))
+    (pad "" np_thru_hole circle (at 0 0) (size 3.5 3.5) (drill 3.5) (layers *.Cu *.Mask))
+  )
+  (footprint "MountingHole:MountingHole_3.5mm" (layer "F.Cu")
     (at 382.2 101)
-    (descr "Mounting Hole 2.2mm, M2")
-    (tags "mounting hole 2.2mm m2")
+    (descr "Mounting Hole 3.5mm, no annular")
+    (tags "mounting hole 3.5mm no annular")
     (property "LCSC part" "")
     (property "Sheetfile" "EnvKB65HS.kicad_sch")
     (property "Sheetname" "")
     (attr exclude_from_pos_files)
-    (fp_text reference "H0" (at 0 -3.2) (layer "F.Fab")
-      (effects (font (size 1 1) (thickness 0.15)))
-    )
-    (fp_text value "SMTWE2020MTJ" (at 0 3.2) (layer "F.Fab")
+    (fp_text reference "H0" (at 0 -4.5) (layer "F.SilkS")
+      (effects (font (size 1 1) (thickness 0.15)))
+    )
+    (fp_text value "C2928180" (at 0 4.5) (layer "F.Fab")
       (effects (font (size 1 1) (thickness 0.15)))
     )
@@
       (effects (font (size 1 1) (thickness 0.15)))
     )
-    (fp_circle (center 0 0) (end 2.2 0) (layer "Cmts.User") (width 0.15) (fill none))
-    (fp_circle (center 0 0) (end 2.45 0) (layer "F.CrtYd") (width 0.05) (fill none))
-    (pad "1" thru_hole circle (at 0 0) (size 6 6) (drill 3.8) (layers *.Cu *.Mask)
-      (net 105 "unconnected-(H0-Pad1)") (pinfunction "1") (pintype "input+no_connect"))
+    (fp_circle (center 0 0) (end 3.5 0) (layer "Cmts.User") (width 0.15) (fill none))
+    (fp_circle (center 0 0) (end 3.75 0) (layer "F.CrtYd") (width 0.05) (fill none))
+    (pad "" np_thru_hole circle (at 0 0) (size 3.5 3.5) (drill 3.5) (layers *.Cu *.Mask))
   )
   (footprint "MX_Only:MXOnly-1U-Hotswap-Modified" (layer "F.Cu")
@@
       (net 75 "Net-(D_58-Pad2)") (pinfunction "ROW") (pintype "passive"))
   )
-  (footprint "Logo:MountingHole_3mm_Pad5.3mm" (layer "F.Cu")
+  (footprint "MountingHole:MountingHole_3.5mm" (layer "F.Cu")
     (at 251.125 183.475)
-    (descr "Mounting Hole 2.2mm, M2")
-    (tags "mounting hole 2.2mm m2")
+    (descr "Mounting Hole 3.5mm, no annular")
+    (tags "mounting hole 3.5mm no annular")
     (property "Sheetfile" "EnvKB65HS.kicad_sch")
     (property "Sheetname" "")
     (attr exclude_from_pos_files)
-    (fp_text reference "H5" (at 0 -3.2) (layer "F.Fab")
-      (effects (font (size 1 1) (thickness 0.15)))
-    )
-    (fp_text value "SMTWE2020MTJ" (at 0 3.2) (layer "F.Fab")
+    (fp_text reference "H5" (at 0 -4.5) (layer "F.SilkS")
+      (effects (font (size 1 1) (thickness 0.15)))
+    )
+    (fp_text value "C2928180" (at 0 4.5) (layer "F.Fab")
       (effects (font (size 1 1) (thickness 0.15)))
     )
@@
       (effects (font (size 1 1) (thickness 0.15)))
     )
-    (fp_circle (center 0 0) (end 2.2 0) (layer "Cmts.User") (width 0.15) (fill none))
-    (fp_circle (center 0 0) (end 2.45 0) (layer "F.CrtYd") (width 0.05) (fill none))
-    (pad "1" thru_hole circle (at 0 0) (size 6 6) (drill 3.8) (layers *.Cu *.Mask)
-      (net 110 "unconnected-(H5-Pad1)") (pinfunction "1") (pintype "input+no_connect"))
-  )
-  (footprint "MX_Only:MXOnly-1U-Hotswap-Modified" (layer "F.Cu")
+    (fp_circle (center 0 0) (end 3.5 0) (layer "Cmts.User") (width 0.15) (fill none))
+    (fp_circle (center 0 0) (end 3.75 0) (layer "F.CrtYd") (width 0.05) (fill none))
+    (pad "" np_thru_hole circle (at 0 0) (size 3.5 3.5) (drill 3.5) (layers *.Cu *.Mask))
+  )
+  (footprint "MX_Only:MXOnly-1U-Hotswap-Modified" (layer "F.Cu")
