File: MainPCB-HOTSWAP/EnvKB65HS.kicad_pcb (KiCad board)
At the start: 2 copper layers, 322.3 x 99.3 mm, 160 parts, among them J1 Conn_01x04, U0 Pico

Commit message: swapped diodes to larger footprint and corrected DRC errors
Parts:
- D_0, D_1, D_10, D_11, D_12, D_13, D_14, D_15, D_16, D_17, D_18, D_19, D_2, D_20, D_21, D_22, D_23, D_24, D_25, D_26, D_27, D_28, D_29, D_3, D_30, D_31, D_32, D_33, D_34, D_35, D_36, D_37, D_38, D_39, D_4, D_40, D_41, D_42, D_43, D_44, D_45, D_46, D_47, D_48, D_49, D_5, D_50, D_51, D_52, D_53, D_54, D_55, D_56, D_57, D_58, D_59, D_6, D_60, D_61, D_62, D_63, D_64, D_65, D_66, D_67, D_68, D_69, D_7, D_70, D_8, D_9: value Diode SOD-323 -> 1n4148; footprint Diode_SMD:D_SOD-323_HandSoldering -> Diode_SMD:D_SOD-123
Routing:
- net row3: track 334.5 -> 322.8 mm, vias 1 -> 0
- net row4: track 347.0 -> 345.8 mm
- net row0: track 355.9 -> 356.9 mm
- net row2: track 312.8 -> 313.7 mm
- net Net-(D_51-Pad2): track 10.5 -> 9.76 mm
- net Net-(D_44-Pad2): track 10.6 -> 9.83 mm
- net Net-(D_69-Pad2): track 8.60 -> 8.00 mm
- net Net-(D_48-Pad2): track 10.6 -> 10.0 mm
- net Net-(D_46-Pad2): track 10.6 -> 10.0 mm
