File: MainPCB/EnvKB65.kicad_pcb (KiCad board)
At the start: 2 copper layers, 320.8 x 99.3 mm, 151 parts, among them U0 Pico

Commit message: various corrections and updated gerbers, bom, cpls
Parts:
- added stab1: Stabilizer, Mounting_Keyboard_Stabilizer:Stabilizer_Cherry_MX_2u, F.Cu at (232.1, 187.7)
- added stab2: Stabilizer, Mounting_Keyboard_Stabilizer:Stabilizer_Cherry_MX_2u, F.Cu at (155.9, 187.7)
- added stab3: Stabilizer, Mounting_Keyboard_Stabilizer:Stabilizer_Cherry_MX_2u, F.Cu at (327.3, 149.6)
- added stab4: Stabilizer, Mounting_Keyboard_Stabilizer:Stabilizer_Cherry_MX_2u, F.Cu at (329.7, 111.5)
- added stab5: Stabilizer, Mounting_Keyboard_Stabilizer:Stabilizer_Cherry_MX_2u, F.Cu at (84.4, 168.7)
- added stab6: Stabilizer, Mounting_Keyboard_Stabilizer:Stabilizer_Cherry_MX_2u, F.Cu at (336.8, 140.1)
- D_0, D_1, D_10, D_11, D_12, D_13, D_14, D_15, D_16, D_17, D_18, D_19, D_2, D_20, D_21, D_22, D_23, D_24, D_25, D_26, D_27, D_28, D_29, D_3, D_30, D_31, D_32, D_33, D_34, D_35, D_36, D_37, D_38, D_39, D_4, D_40, D_41, D_42, D_43, D_44, D_45, D_46, D_47, D_48, D_49, D_5, D_50, D_51, D_52, D_53, D_54, D_55, D_56, D_57, D_58, D_59, D_6, D_60, D_61, D_62, D_63, D_64, D_65, D_66, D_67, D_68, D_69, D_7, D_70, D_8, D_9: value Diode SOD-323 -> 1n4148 sod-323
- K_0, K_1, K_10, K_11, K_12, K_15, K_16, K_17, K_18, K_19, K_2, K_20, K_21, K_22, K_23, K_24, K_25, K_26, K_3, K_30, K_31, K_32, K_33, K_34, K_35, K_36, K_37, K_38, K_39, K_4, K_40, K_41, K_45, K_46, K_47, K_48, K_49, K_5, K_50, K_51, K_52, K_53, K_54, K_55, K_57, K_58, K_59, K_6, K_66, K_67, K_68, K_69, K_7, K_70, K_71, K_72, K_8, K_9: value KEYSW -> MX Switch
- K_13: value KEYSW -> MX Switch; footprint MX_Only:MXOnly-2U-NoLED -> MX_Only:MXOnly-1U-NoLED
- K_14, K_27: value KEYSW -> MX Switch; footprint MX_Only:MXOnly-1.5U-NoLED -> MX_Only:MXOnly-1U-NoLED
- K_28, K_43: value KEYSW -> MX Switch; footprint MX_Only:MXOnly-2.25U-NoLED -> MX_Only:MXOnly-1U-NoLED
- K_29, K_56, K_64: value KEYSW -> MX Switch; footprint MX_Only:MXOnly-1.75U-NoLED -> MX_Only:MXOnly-1U-NoLED
- K_42: value KEYSW -> MX Switch; footprint MX_Only:MXOnly-ISO-ROTATED-ReversedStabilizers-NoLED -> MX_Only:MXOnly-1U-NoLED
- K_44, K_60, K_61, K_62: value KEYSW -> MX Switch; footprint MX_Only:MXOnly-1.25U-NoLED -> MX_Only:MXOnly-1U-NoLED
- K_63, K_65: value KEYSW -> MX Switch; footprint MX_Only:MXOnly-2.25U-ReversedStabilizers-NoLED -> MX_Only:MXOnly-1U-NoLED
- moved D_57 2.25 mm to (368.7, 170.3)
- moved D_56 2.19 mm to (366.4, 170.3)
- turned K_27 to -90 degrees
- turned K_42 to 90 degrees
Connections:
- U0 pad 30: Net-(U0-Pad30) -> unconnected-(U0-Pad30)
- U0 pad 35: Net-(U0-Pad35) -> unconnected-(U0-Pad35)
- U0 pad 36: Net-(U0-Pad36) -> unconnected-(U0-Pad36)
- U0 pad 37: Net-(U0-Pad37) -> unconnected-(U0-Pad37)
- U0 pad 39: Net-(U0-Pad39) -> unconnected-(U0-Pad39)
- U0 pad 40: Net-(U0-Pad40) -> unconnected-(U0-Pad40)
Routing:
- net Net-(D_27-Pad2): track 24.9 -> 35.6 mm
- net Net-(D_66-Pad2): track 15.8 -> 8.22 mm
- net col14: track 140.1 -> 133.7 mm
- net col0: track 389.0 -> 385.6 mm
- net Net-(D_56-Pad2): track 11.2 -> 8.77 mm
- net Net-(D_57-Pad2): track 17.7 -> 15.5 mm
- net Net-(D_41-Pad2): track 31.4 -> 33.6 mm
- net Net-(D_42-Pad2): track 22.7 -> 20.7 mm
- net col12: track 174.9 -> 173.0 mm
- net row1: track 324.2 -> 322.5 mm, vias 0 -> 2
- net col10: track 206.6 -> 204.9 mm
- net col2: track 326.1 -> 324.5 mm
- net Net-(D_40-Pad2): track 14.8 -> 13.2 mm
- net Net-(D_70-Pad2): track 16.7 -> 15.2 mm
- net col6: track 275.2 -> 274.0 mm
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Other:
- net class Default removed
- board text added: "http://github.com/Envious-Data/Env-KB65M https://github.com/Envious-Data/EnvKB-QMK https://envious.design/firmwares/"
- board text removed: "http://github.com/Envious-Data/Env-KB65M"
- board text removed: "https://github.com/Envious-Data/Env-KB65M"

Commit message: swapped diodes to larger footprint and corrected DRC errors
Parts:
- D_0, D_1, D_10, D_11, D_12, D_13, D_14, D_15, D_16, D_17, D_18, D_19, D_2, D_20, D_21, D_22, D_23, D_24, D_25, D_26, D_27, D_28, D_29, D_3, D_30, D_31, D_32, D_33, D_34, D_35, D_36, D_37, D_38, D_39, D_4, D_40, D_41, D_42, D_43, D_44, D_45, D_46, D_47, D_48, D_49, D_5, D_50, D_51, D_52, D_53, D_54, D_55, D_56, D_57, D_58, D_59, D_6, D_60, D_61, D_62, D_63, D_64, D_65, D_66, D_67, D_68, D_69, D_7, D_70, D_8, D_9: value 1n4148 sod-323 -> 1n4148; footprint Diode_SMD:D_SOD-323_HandSoldering -> Diode_SMD:D_SOD-123
Routing:
- net row2: track 314.4 -> 316.2 mm
- net row4: track 348.2 -> 347.7 mm
