File: MainPCB/EnvKB65.kicad_sch (KiCad schematic)
At the start: 157 parts, among them U0 Pico

Commit message: swapped diodes to larger footprint and corrected DRC errors
Parts:
- D_0, D_1, D_10, D_11, D_12, D_13, D_14, D_15, D_16, D_17, D_18, D_19, D_2, D_20, D_21, D_22, D_23, D_24, D_25, D_26, D_27, D_28, D_29, D_3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: value 1n4148 sod-323 -> 1n4148; footprint Diode_SMD:D_SOD-323_HandSoldering -> Diode_SMD:D_SOD-123
